Commit message: added robot mesh

File: scitos_description/urdf/scitos.urdf (robot description, URDF)
Before this commit: robot scitosA5, 7 links, 6 joints
Links:
- link base_link: geometry collision cylinder length=0.6 radius=0.2; visual mesh filename=package://scitos_description/meshes/scitos.dae

Commit message: update urdf to include xtion and pantilt

File: scitos_description/urdf/scitos.urdf (robot description, URDF)
Before this commit: robot scitosA5, 7 links, 6 joints
Links:
- removed link camera_link
- removed link kinect_link
- removed link ptz_link
- removed link ptz_mid_link
- added link head_xtion_link, mass 1.0; collision box size=0.001 0.001 0.001; visual mesh filename=package://scitos_description/meshes/xtion.dae
- added link ptu_mount, mass 1; collision box size=.03 .27 .004; visual box size=.06 .27 0.004
- added link ptu_pan_motor, mass 1; collision box size=0.04 .07 .05; visual box size=0.04 .07 .05
- added link ptu_tilt_motor, mass 1; collision box size=0.04 .04 .06; visual box size=0.04 .04 .06
- link base_footprint: geometry collision box size=0.001 0.001 0.001; visual mesh filename=package://scitos_description/meshes/scitos.dae
- link base_link: geometry collision cylinder length=0.6 radius=0.2; visual box size=0 0 0
Joints:
- removed joint camera_joint
- removed joint kinect_joint
- removed joint ptz_y_joint
- removed joint ptz_z_joint
- added joint head_xtion_joint: type fixed, parent ptu_mount, child head_xtion_link, origin xyz=0 0 0.03 rpy=3.14 0 0, axis 0 0 1
- added joint pan: type continuous, parent ptu_pan_motor, child ptu_tilt_motor, origin xyz=0 0 .055, axis 0 0 1
- added joint pantilt_joint: type fixed, parent base_link, child ptu_pan_motor, origin xyz=0.0 0.0 1.534 rpy=0 0 0
- added joint tilt: type continuous, parent ptu_tilt_motor, child ptu_mount, origin xyz=0 0 .043, axis 0 -1 0
