Commit message: using the new and accurate ptu transforms and model

File: scitos_description/urdf/scitos.xacro (robot description, xacro)
@@ -18,4 +18,25 @@
     <color rgba="0.65 0.65 0.65 1.0"/>
   </material>
+  <!-- base_footprint : a fictional link that is on the floor plane, needed for move_base -->
+  <link name="base_footprint">
+    <inertial>
+      <mass value="1.0"/>
+      <origin xyz="0 0 0"/>
+      <inertia ixx="0.01" ixy="0.0" ixz="0.0" iyy="0.01" iyz="0.0" izz="0.01"/>
+    </inertial>
+    <visual>
+      <origin rpy="0 0 0" xyz="0 0 0"/>
+      <geometry>
+        <box size="0 0 0"/>
+      </geometry>
+      <material name="Red"/>
+    </visual>
+    <collision>
+      <origin rpy="0 0 0" xyz="0 0 0"/>
+      <geometry>
+        <box size="0 0 0"/>
+      </geometry>
+    </collision>
+  </link>
   <!-- Base link is the actual robot body -->
   <link name="base_link">
@@ -26,5 +47,5 @@
     </inertial>
     <visual>
-      <origin rpy="0 0 0" xyz="0 0 0.0"/>
+      <origin rpy="0 0 0" xyz="0 0 0"/>
       <geometry>
 	<mesh filename="package://scitos_description/meshes/scitos.dae"/>
@@ -35,25 +56,4 @@
       <geometry>
         <cylinder length="0.6" radius="0.2"/>
-      </geometry>
-    </collision>
-  </link>
-  <!-- base_footprint : a fictional link that is on the floor plane, needed for move_base -->
-  <link name="base_footprint">
-    <inertial>
-      <mass value="1.0"/>
-      <origin xyz="0 0 0"/>
-      <inertia ixx="0.01" ixy="0.0" ixz="0.0" iyy="0.01" iyz="0.0" izz="0.01"/>
-    </inertial>
-    <visual>
-      <origin rpy="0 0 0" xyz="0 0 0"/>
-      <geometry>
-        <box size="0 0 0"/>
-      </geometry>
-      <material name="Red"/>
-    </visual>
-    <collision>
-      <origin rpy="0 0 0" xyz="0 0 0.071"/>
-      <geometry>
-        <box size="0 0 0"/>
       </geometry>
     </collision>
@@ -61,7 +61,7 @@
   <!-- Base footprint -> base_link -->
   <joint name="base_footprint_joint" type="fixed">
-    <origin rpy="0 0 0" xyz="0 0 0.051"/>
+    <origin rpy="0 0 0" xyz="0 0 0.021"/>
+    <parent link="base_footprint"/>
     <child link="base_link"/>
-    <parent link="base_footprint"/>
   </joint>
   <!-- base_link -> base_laser_link -->
@@ -77,7 +77,13 @@
     <inertial>
       <mass value="0.001"/>
-      <origin rpy="0 0 0" xyz="0 0 0"/>
+      <origin rpy="0 0 0" xyz="0 0 0.075"/>
       <inertia ixx="0.0001" ixy="0" ixz="0" iyy="0.000001" iyz="0" izz="0.0001"/>
     </inertial>
+    <visual>
+      <origin rpy="0 0 0" xyz="0 0 0.075"/>
+      <geometry>
+	<cylinder length="0.15" radius="0.04"/>
+      </geometry>
+    </visual>
   </link>
   <!-- Pan-Tilt lower motor -->
@@ -89,7 +95,7 @@
     </inertial>
     <visual>
-      <origin xyz="0 -0.015 0"/>
-      <geometry>
-        <box size="0.04 .07 .05"/>
+      <origin xyz="0 0 0" rpy="0 0 0"/>
+      <geometry>
+	<mesh filename="package://scitos_description/meshes/pantil0_1.dae"/>
       </geometry>
       <material name="Black"/>
@@ -117,7 +123,7 @@
     </inertial>
     <visual>
-      <origin/>
-      <geometry>
-        <box size="0.04 .04 .06"/>
+      <origin xyz="0 0 0" rpy="0 0 0"/>
+      <geometry>
+	<mesh filename="package://scitos_description/meshes/pantil1_1.dae"/>
       </geometry>
       <material name="Black"/>
@@ -132,6 +138,6 @@
   <!-- pan joint -->
   <joint name="pan" type="continuous">
-    <origin xyz="0 0 .055"/>
-    <axis xyz="0 0 1"/>
+    <origin xyz="0 0 0.04572" rpy="1.57 0 0"/>
+    <axis xyz="0 1 0"/>
     <parent link="ptu_pan_motor"/>
     <child link="ptu_tilt_motor"/>
@@ -145,7 +151,7 @@
     </inertial>
     <visual>
-      <origin/>
-      <geometry>
-        <box size=" .06 .27 0.004 "/>
+      <origin xyz="0 0 0" rpy="0 0 0"/>
+      <geometry>
+	<mesh filename="package://scitos_description/meshes/pantil2_1.dae"/>
       </geometry>
       <material name="Aluminium"/>
@@ -160,6 +166,6 @@
   <!-- tilt joint -->
   <joint name="tilt" type="continuous">
-    <origin xyz="0 0 .043"/>
-    <axis xyz="0 -1 0"/>
+    <origin xyz="0 0.045974 0" rpy="-1.57 0 0"/>
+    <axis xyz="0 1 0"/>
     <parent link="ptu_tilt_motor"/>
     <child link="ptu_mount"/>

File: scitos_description/urdf/scitos_calibration.xacro (robot description, xacro)
@@ -5,12 +5,12 @@
   <property name="front_laser_scan_trans_x" value="0.30" />
   <property name="front_laser_scan_trans_y" value="0" />
-  <property name="front_laser_scan_trans_z" value="0.386" />
+  <property name="front_laser_scan_trans_z" value="0.365" />
   <property name="front_laser_scan_rot_x" value="0.0" />
   <property name="front_laser_scan_rot_y" value="0.0" />
   <property name="front_laser_scan_rot_z" value="0.0" />
   <!-- the pan tilt unit -->
-  <property name="pan_tilt_base_plate_trans_x" value="0.0" />
+  <property name="pan_tilt_base_plate_trans_x" value="0.075" />
   <property name="pan_tilt_base_plate_trans_y" value="0.0" />
-  <property name="pan_tilt_base_plate_trans_z" value="1.585" />
+  <property name="pan_tilt_base_plate_trans_z" value="1.5183" />
   <property name="pan_tilt_base_plate_rot_x" value="0.0" />
   <property name="pan_tilt_base_plate_rot_y" value="0.0" />

Commit message: improve camera position, use new link model.

File: scitos_description/urdf/scitos.xacro (robot description, xacro)
@@ -143,6 +143,6 @@
     <child link="ptu_tilt_motor"/>
   </joint>
-  <!-- the top aluminium plate on the ptu unit -->
-  <link name="ptu_mount">
+  <!-- the top pantilt hinge bracket that joints the tilt motor to the aluminium plate -->
+  <link name="ptu_hinge">
     <inertial>
       <mass value="1"/>
@@ -155,5 +155,4 @@
 	<mesh filename="package://scitos_description/meshes/pantil2_1.dae"/>
       </geometry>
-      <material name="Aluminium"/>
     </visual>
     <collision>
@@ -169,4 +168,31 @@
     <axis xyz="0 1 0"/>
     <parent link="ptu_tilt_motor"/>
+    <child link="ptu_hinge"/>
+  </joint>
+  <!-- ptu_mount: the top aluminium plate on the ptu unit -->
+  <link name="ptu_mount">
+    <inertial>
+      <mass value="1"/>
+      <inertia ixx="100" ixy="0" ixz="0" iyy="100" iyz="0" izz="100"/>
+      <origin/>
+    </inertial>
+    <visual>
+      <origin xyz="0 0 0" rpy="0 0 0"/>
+      <geometry>
+	<mesh filename="package://scitos_description/meshes/pantil3_1.dae"/>
+      </geometry>
+      <material name="Aluminium"/>
+    </visual>
+    <collision>
+      <origin/>
+      <geometry>
+        <box size=" .03 .27 .004"/>
+      </geometry>
+    </collision>
+  </link>
+  <!-- ptu_hing -> ptu_mount -->
+  <joint name="hinge_to_mount" type="fixed">
+    <origin xyz="0 0 0.039116" rpy="0 0 0"/>
+    <parent link="ptu_hinge"/>
     <child link="ptu_mount"/>
   </joint>

File: scitos_description/urdf/scitos_calibration.xacro (robot description, xacro)
@@ -17,5 +17,5 @@
   <property name="pan_tilt_base_plate_rot_z" value="0.0" />
   <!-- the head_xtion relative to the ptu top mount frame -->
-  <property name="head_xtion_trans_x" value="0.0" />
+  <property name="head_xtion_trans_x" value="0.015" />
   <property name="head_xtion_trans_y" value="0.0" />
   <property name="head_xtion_trans_z" value="0.03" />

Commit message: tidying mesh file names and removing old meshes

File: scitos_description/urdf/scitos.xacro (robot description, xacro)
@@ -97,5 +97,5 @@
       <origin xyz="0 0 0" rpy="0 0 0"/>
       <geometry>
-	<mesh filename="package://scitos_description/meshes/pantil0_1.dae"/>
+	<mesh filename="package://scitos_description/meshes/pantilt0.dae"/>
       </geometry>
       <material name="Black"/>
@@ -125,5 +125,5 @@
       <origin xyz="0 0 0" rpy="0 0 0"/>
       <geometry>
-	<mesh filename="package://scitos_description/meshes/pantil1_1.dae"/>
+	<mesh filename="package://scitos_description/meshes/pantilt1.dae"/>
       </geometry>
       <material name="Black"/>
@@ -153,5 +153,5 @@
       <origin xyz="0 0 0" rpy="0 0 0"/>
       <geometry>
-	<mesh filename="package://scitos_description/meshes/pantil2_1.dae"/>
+	<mesh filename="package://scitos_description/meshes/pantilt2.dae"/>
       </geometry>
     </visual>
@@ -180,5 +180,5 @@
       <origin xyz="0 0 0" rpy="0 0 0"/>
       <geometry>
-	<mesh filename="package://scitos_description/meshes/pantil3_1.dae"/>
+	<mesh filename="package://scitos_description/meshes/pantilt3.dae"/>
       </geometry>
       <material name="Aluminium"/>

Commit message: initial transforms in place

File: scitos_description/urdf/scitos.xacro (robot description, xacro)
@@ -18,4 +18,31 @@
     <color rgba="0.65 0.65 0.65 1.0"/>
   </material>
+  <material name="white">
+	<color rgba="1 1 1 1" />
+  </material>
+  <material name="black">
+	<color rgba="0 0 0 1" />
+  </material>
+  <material name="red">
+	<color rgba="1 0 0 1" />
+  </material>
+  <material name="green">
+	<color rgba="0 1 0 1" />
+  </material>
+  <material name="blue">
+	<color rgba="0 0 1 1" />
+  </material>
+  <material name="yellow">
+	<color rgba="1 1 0 1" />
+  </material>
+  <material name="darkgray">
+	<color rgba="0.3 0.3 0.3 1" />
+  </material>
+  <material name="gray">
+	<color rgba="0.7 0.7 0.7 1" />
+  </material>
+  <material name="glass">
+	<color rgba="1 1 1 0.2" />
+  </material>
   <!-- base_footprint : a fictional link that is on the floor plane, needed for move_base -->
   <link name="base_footprint">
@@ -49,5 +76,6 @@
       <origin rpy="0 0 0" xyz="0 0 0"/>
       <geometry>
-	<mesh filename="package://scitos_description/meshes/scitos.dae"/>
+<!--	<mesh filename="package://scitos_description/meshes/scitos.dae"/> -->
+        <cylinder length="0.0" radius="0.2"/>
       </geometry>
     </visual>
@@ -225,3 +253,94 @@
     <child link="head_xtion_link"/>
   </joint>
+  <!-- HEAD -->
+  <joint name="HMIToHeadBase" type="fixed">
+	<parent link="base_link" />
+	<child link="HeadBaseFrame" />
+	<origin xyz="0 0 0.7375" />
+  </joint>
+  <link name="HeadSwivelFrame">
+	<visual>
+	  <geometry>
+		<cylinder length="0.1" radius="0.05" />
+	  </geometry>
+	  <material name="gray" />
+	</visual>
+  </link>
+  <joint name="HeadPan" type="continuous">
+	<parent link="HeadBaseFrame" />
+	<child link="HeadSwivelFrame" />
+	<axis xyz="0 0 1" />
+  </joint>
+  <link name="HeadFrame">
+	<visual>
+	  <geometry>
+		<box size="0.175 0.19 0.07" />
+	  </geometry>
+	  <origin xyz="0 0 0.02" rpy="0 0 0" />
+	  <material name="gray" />
+	</visual>
+  </link>
+  <joint name="HeadTilt" type="continuous">
+	<parent link="HeadSwivelFrame" />
+	<child link="HeadFrame" />
+	<axis xyz="0 1 0" />
+  </joint>
+  <link name="LeftEyeFrame">
+	<visual>
+	  <geometry>
+		<sphere radius="0.025" />
+	  </geometry>
+	  <material name="white" />
+	</visual>
+  </link>
+  <joint name="HeadToLeftEyeBase" type="fixed">
+	<parent link="HeadFrame" />
+	<child link="LeftEyeBaseFrame" />
+	<origin xyz="0.08 0.05 0.02" />
+  </joint>
+  <joint name="EyesTilt" type="continuous">
+	<parent link="LeftEyeBaseFrame" />
+	<child link="LeftEyeSwivelFrame" />
+	<axis xyz="0 1 0" />
+  </joint>
+  <joint name="EyesPan" type="continuous">
+	<parent link="LeftEyeSwivelFrame" />
+	<child link="LeftEyeFrame" />
+	<axis xyz="0 0 1" />
+  </joint>
+  <link name="RightEyeFrame">
+	<visual>
+	  <geometry>
+		<sphere radius="0.025" />
+	  </geometry>
+	  <material name="white" />
+	</visual>
+  </link>
+  <joint name="HeadToRightEyeBase" type="fixed">
+	<parent link="HeadFrame" />
+	<child link="RightEyeBaseFrame" />
+	<origin xyz="0.08 -0.05 0.02" />
+  </joint>
+  <joint name="RightEyeBaseToRightEyeSwivel" type="continuous">
+	<parent link="RightEyeBaseFrame" />
+	<child link="RightEyeSwivelFrame" />
+	<axis xyz="0 1 0" />
+  </joint>
+  <joint name="RightEyeSwivelToRightEye" type="continuous">
+	<parent link="RightEyeSwivelFrame" />
+	<child link="RightEyeFrame" />
+	<axis xyz="0 0 1" />
+  </joint>
+  <link name="HeadBaseFrame">
+	<visual>
+	  <geometry>
+		<sphere radius="0.15" />
+	  </geometry>
+	  <material name="glass"/>
+	</visual>
+  </link>
+  <link name="RightEyeBaseFrame" />
+  <link name="LeftEyeBaseFrame" />
+  <link name="RightEyeSwivelFrame" />
+  <link name="LeftEyeSwivelFrame" />
 </robot>

Commit message: added xtion frames to urdf

File: scitos_description/urdf/scitos.xacro (robot description, xacro)
@@ -225,3 +225,32 @@
     <child link="head_xtion_link"/>
   </joint>
+  <!-- xtion camera internal frames (these moved from openni_launch/kinect_frames.launch) -->
+  <link name="head_xtion_depth_frame" />
+  <link name="head_xtion_rgb_frame" />
+  <link name="head_xtion_depth_optical_frame" />
+  <link name="head_xtion_rgb_optical_frame" />
+  <joint name="head_xtion_base_link" type="fixed">
+        <origin xyz="0 -0.02  0"
+				rpy="0 0 0" />
+		<parent link="head_xtion_link" />
+		<child link="head_xtion_depth_frame" />
+  </joint>
+  <joint name="head_xtion_base_link2" type="fixed" >
+        <origin xyz="0 -0.045  0"
+				rpy="0 0 0" />
+		<parent link="head_xtion_link" />
+		<child link="head_xtion_rgb_frame" />
+  </joint>
+  <joint name="head_xtion_base_link3"  type="fixed">
+        <origin xyz="0 0 0"
+				rpy="-3.14 0 -3.14" />
+		<parent link="head_xtion_depth_frame" />
+		<child link="head_xtion_depth_optical_frame" />
+  </joint>
+  <joint name="head_xtion_base_link4"  type="fixed">
+        <origin xyz="0 0 0"
+				rpy="-3.14 0 -3.14" />
+		<parent link="head_xtion_rgb_frame" />
+		<child link="head_xtion_rgb_optical_frame" />
+  </joint>
 </robot>

Commit message: adding new model and xtion frames

File: scitos_description/urdf/scitos.xacro (robot description, xacro)
@@ -49,5 +49,5 @@
       <origin rpy="0 0 0" xyz="0 0 0"/>
       <geometry>
-	<mesh filename="package://scitos_description/meshes/scitos.dae"/>
+	<mesh filename="package://scitos_description/meshes/scitos_1.dae"/>
       </geometry>
     </visual>
@@ -87,4 +87,24 @@
     </visual>
   </link>
+  <!-- base_halo is the metal frame that the ptu sit on top of-->
+  <link name="base_halo">
+    <visual>
+      <origin rpy="0 0 0" xyz="0 0 0"/>
+      <geometry>
+	<mesh filename="package://scitos_description/meshes/head_frame.dae"/>
+      </geometry>
+    </visual>
+    <collision>
+      <origin rpy="0 0 0" xyz="0 0 0.25"/>
+      <geometry>
+        <cylinder length="0.5" radius="0.25"/>
+      </geometry>
+    </collision>
+  </link>
+  <joint name="base_halo_joint" type="fixed" >
+    <origin  xyz="0 0 0" rpy="0 0 0"/>
+    <parent link="base_link" />
+    <child link="base_halo" />
+  </joint>
   <!-- Pan-Tilt lower motor -->
   <link name="ptu_pan_motor">
@@ -232,25 +252,25 @@
   <joint name="head_xtion_base_link" type="fixed">
         <origin xyz="0 -0.02  0"
-				rpy="0 0 0" />
-		<parent link="head_xtion_link" />
-		<child link="head_xtion_depth_frame" />
+		rpy="0 0 0" />
+	<parent link="head_xtion_link" />
+	<child link="head_xtion_depth_frame" />
   </joint>
   <joint name="head_xtion_base_link2" type="fixed" >
         <origin xyz="0 -0.045  0"
-				rpy="0 0 0" />
-		<parent link="head_xtion_link" />
-		<child link="head_xtion_rgb_frame" />
+		rpy="0 0 0" />
+	<parent link="head_xtion_link" />
+	<child link="head_xtion_rgb_frame" />
   </joint>
   <joint name="head_xtion_base_link3"  type="fixed">
         <origin xyz="0 0 0"
-				rpy="-3.14 0 -3.14" />
-		<parent link="head_xtion_depth_frame" />
-		<child link="head_xtion_depth_optical_frame" />
+		rpy="-1.57 0 1.57" />
+	<parent link="head_xtion_depth_frame" />
+	<child link="head_xtion_depth_optical_frame" />
   </joint>
   <joint name="head_xtion_base_link4"  type="fixed">
         <origin xyz="0 0 0"
-				rpy="-3.14 0 -3.14" />
-		<parent link="head_xtion_rgb_frame" />
-		<child link="head_xtion_rgb_optical_frame" />
+		rpy="-1.57 0 1.57" />
+	<parent link="head_xtion_rgb_frame" />
+	<child link="head_xtion_rgb_optical_frame" />
   </joint>
 </robot>

Commit message: using new model, adding in head transformations..

File: scitos_description/urdf/scitos.xacro (robot description, xacro)
@@ -108,8 +108,9 @@
     </inertial>
     <visual>
-      <origin rpy="0 0 0" xyz="0 0 0.075"/>
-      <geometry>
-	<cylinder length="0.15" radius="0.04"/>
-      </geometry>
+      <origin rpy="0 0 0" xyz="0 0 -0.09"/>
+      <geometry>
+		<cylinder length="0.18" radius="0.04"/>
+      </geometry>
+	  <material name="yellow" />
     </visual>
   </link>
@@ -273,10 +274,18 @@
   </joint>
   <!-- HEAD -->
-  <joint name="HMIToHeadBase" type="fixed">
+  <link name="head_base_frame">
+	<visual>
+	  <geometry>
+		<sphere radius="0.15" />
+	  </geometry>
+	  <material name="glass"/>
+	</visual>
+  </link>
+  <joint name="base_link_to_head" type="fixed">
 	<parent link="base_link" />
-	<child link="HeadBaseFrame" />
-	<origin xyz="0 0 0.7375" />
-  </joint>
-  <link name="HeadSwivelFrame">
+	<child link="head_base_frame" />
+	<origin xyz="-0.075 0 1.32" />
+  </joint>
+  <link name="head_swivel_frame">
 	<visual>
 	  <geometry>
@@ -287,9 +296,9 @@
   </link>
   <joint name="HeadPan" type="continuous">
-	<parent link="HeadBaseFrame" />
-	<child link="HeadSwivelFrame" />
+	<parent link="head_base_frame" />
+	<child link="head_swivel_frame" />
 	<axis xyz="0 0 1" />
   </joint>
-  <link name="HeadFrame">
+  <link name="head_frame">
 	<visual>
 	  <geometry>
@@ -301,9 +310,9 @@
   </link>
   <joint name="HeadTilt" type="continuous">
-	<parent link="HeadSwivelFrame" />
-	<child link="HeadFrame" />
+	<parent link="head_swivel_frame" />
+	<child link="head_frame" />
 	<axis xyz="0 1 0" />
   </joint>
-  <link name="LeftEyeFrame">
+  <link name="left_eye_frame">
 	<visual>
 	  <geometry>
@@ -314,19 +323,19 @@
   </link>
   <joint name="HeadToLeftEyeBase" type="fixed">
-	<parent link="HeadFrame" />
-	<child link="LeftEyeBaseFrame" />
+	<parent link="head_frame" />
+	<child link="left_eye_base_frame" />
 	<origin xyz="0.08 0.05 0.02" />
   </joint>
   <joint name="EyesTilt" type="continuous">
-	<parent link="LeftEyeBaseFrame" />
-	<child link="LeftEyeSwivelFrame" />
+	<parent link="left_eye_base_frame" />
+	<child link="left_eye_swivel_frame" />
 	<axis xyz="0 1 0" />
   </joint>
   <joint name="EyesPan" type="continuous">
-	<parent link="LeftEyeSwivelFrame" />
-	<child link="LeftEyeFrame" />
+	<parent link="left_eye_swivel_frame" />
+	<child link="left_eye_frame" />
 	<axis xyz="0 0 1" />
   </joint>
-  <link name="RightEyeFrame">
+  <link name="right_eye_frame">
 	<visual>
 	  <geometry>
@@ -336,32 +345,25 @@
 	</visual>
   </link>
-  <joint name="HeadToRightEyeBase" type="fixed">
-	<parent link="HeadFrame" />
-	<child link="RightEyeBaseFrame" />
+  <joint name="head_to_right_eye_base" type="fixed">
+	<parent link="head_frame" />
+	<child link="right_eye_base_frame" />
 	<origin xyz="0.08 -0.05 0.02" />
   </joint>
   <joint name="RightEyeBaseToRightEyeSwivel" type="continuous">
-	<parent link="RightEyeBaseFrame" />
-	<child link="RightEyeSwivelFrame" />
+	<parent link="right_eye_base_frame" />
+	<child link="right_eye_swivel_frame" />
 	<axis xyz="0 1 0" />
   </joint>
   <joint name="RightEyeSwivelToRightEye" type="continuous">
-	<parent link="RightEyeSwivelFrame" />
-	<child link="RightEyeFrame" />
+	<parent link="right_eye_swivel_frame" />
+	<child link="right_eye_frame" />
 	<axis xyz="0 0 1" />
   </joint>
-  <link name="HeadBaseFrame">
-	<visual>
-	  <geometry>
-		<sphere radius="0.15" />
-	  </geometry>
-	  <material name="glass"/>
-	</visual>
-  </link>
-  <link name="RightEyeBaseFrame" />
-  <link name="LeftEyeBaseFrame" />
-  <link name="RightEyeSwivelFrame" />
-  <link name="LeftEyeSwivelFrame" />
+  <link name="right_eye_base_frame" />
+  <link name="left_eye_base_frame" />
+  <link name="right_eye_swivel_frame" />
+  <link name="left_eye_swivel_frame" />
   <!-- xtion camera internal frames (these moved from openni_launch/kinect_frames.launch) -->
+<!-- in need of fixing...
   <link name="head_xtion_depth_frame" />
   <link name="head_xtion_rgb_frame" />
@@ -392,3 +394,4 @@
 	<child link="head_xtion_rgb_optical_frame" />
   </joint>
+-->
 </robot>

File: scitos_description/urdf/scitos_calibration.xacro (robot description, xacro)
@@ -3,5 +3,5 @@
   <!-- calibration params -->
   <!-- front laser -->
-  <property name="front_laser_scan_trans_x" value="0.30" />
+  <property name="front_laser_scan_trans_x" value="0.07" />
   <property name="front_laser_scan_trans_y" value="0" />
   <property name="front_laser_scan_trans_z" value="0.365" />
@@ -10,5 +10,5 @@
   <property name="front_laser_scan_rot_z" value="0.0" />
   <!-- the pan tilt unit -->
-  <property name="pan_tilt_base_plate_trans_x" value="0.075" />
+  <property name="pan_tilt_base_plate_trans_x" value="-0.075" />
   <property name="pan_tilt_base_plate_trans_y" value="0.0" />
   <property name="pan_tilt_base_plate_trans_z" value="1.5183" />
