Commit message: removed inertia sections; added xtion frames for head camera

File: scitos_description/urdf/scitos.xacro (robot description, xacro)
@@ -47,9 +47,4 @@
   <!-- base_footprint : a fictional link that is on the floor plane, needed for move_base -->
   <link name="base_footprint">
-    <inertial>
-      <mass value="1.0"/>
-      <origin xyz="0 0 0"/>
-      <inertia ixx="0.01" ixy="0.0" ixz="0.0" iyy="0.01" iyz="0.0" izz="0.01"/>
-    </inertial>
     <visual>
       <origin rpy="0 0 0" xyz="0 0 0"/>
@@ -68,9 +63,4 @@
   <!-- Base link is the actual robot body -->
   <link name="base_link">
-    <inertial>
-      <mass value="74.5"/>
-      <origin xyz="-0.061 0.0 0.1465"/>
-      <inertia ixx="5.652232699207" ixy="-0.009719934438" ixz="1.293988226423" iyy="5.669473158652" iyz="-0.007379583694" izz="3.683196351726"/>
-    </inertial>
     <visual>
       <origin rpy="0 0 0" xyz="0 0 0"/>
@@ -102,9 +92,4 @@
   <!-- the laser -->
   <link name="base_laser_link" type="laser">
-    <inertial>
-      <mass value="0.001"/>
-      <origin rpy="0 0 0" xyz="0 0 0.075"/>
-      <inertia ixx="0.0001" ixy="0" ixz="0" iyy="0.000001" iyz="0" izz="0.0001"/>
-    </inertial>
     <visual>
       <origin rpy="0 0 0" xyz="0 0 -0.09"/>
@@ -137,9 +122,4 @@
   <!-- Pan-Tilt lower motor -->
   <link name="ptu_pan_motor">
-    <inertial>
-      <mass value="1"/>
-      <inertia ixx="100" ixy="0" ixz="0" iyy="100" iyz="0" izz="100"/>
-      <origin/>
-    </inertial>
     <visual>
       <origin xyz="0 0 0" rpy="0 0 0"/>
@@ -165,9 +145,4 @@
   <!-- pantilt upper motor -->
   <link name="ptu_tilt_motor">
-    <inertial>
-      <mass value="1"/>
-      <inertia ixx="100" ixy="0" ixz="0" iyy="100" iyz="0" izz="100"/>
-      <origin/>
-    </inertial>
     <visual>
       <origin xyz="0 0 0" rpy="0 0 0"/>
@@ -193,9 +168,4 @@
   <!-- the top pantilt hinge bracket that joints the tilt motor to the aluminium plate -->
   <link name="ptu_hinge">
-    <inertial>
-      <mass value="1"/>
-      <inertia ixx="100" ixy="0" ixz="0" iyy="100" iyz="0" izz="100"/>
-      <origin/>
-    </inertial>
     <visual>
       <origin xyz="0 0 0" rpy="0 0 0"/>
@@ -220,9 +190,4 @@
   <!-- ptu_mount: the top aluminium plate on the ptu unit -->
   <link name="ptu_mount">
-    <inertial>
-      <mass value="1"/>
-      <inertia ixx="100" ixy="0" ixz="0" iyy="100" iyz="0" izz="100"/>
-      <origin/>
-    </inertial>
     <visual>
       <origin xyz="0 0 0" rpy="0 0 0"/>
@@ -247,9 +212,4 @@
   <!-- xtion camera on head -->
   <link name="head_xtion_link">
-    <inertial>
-      <mass value="1.0"/>
-      <origin xyz="0 0 0"/>
-      <inertia ixx="0.01" ixy="0.0" ixz="0.0" iyy="0.01" iyz="0.0" izz="0.01"/>
-    </inertial>
     <visual>
       <origin rpy="0 0 0" xyz="0 0 0"/>
@@ -365,33 +325,31 @@
   <link name="left_eye_swivel_frame" />
   <!-- xtion camera internal frames (these moved from openni_launch/kinect_frames.launch) -->
-<!-- in need of fixing...
-  <link name="head_xtion_depth_frame" />
-  <link name="head_xtion_rgb_frame" />
-  <link name="head_xtion_depth_optical_frame" />
-  <link name="head_xtion_rgb_optical_frame" />
-  <joint name="head_xtion_base_link" type="fixed">
-        <origin xyz="0 -0.02  0"
-		rpy="0 0 0" />
-	<parent link="head_xtion_link" />
-	<child link="head_xtion_depth_frame" />
+  <link name="head_xtion_depth_frame"/>
+  <link name="head_xtion_rgb_frame"/>
+  <link name="head_xtion_depth_optical_frame"/>
+  <link name="head_xtion_rgb_optical_frame"/>
+  <joint name="head_xtion_base_link" type="fixed" >
+    <origin rpy="0 0 0"
+            xyz="0 -0.02 0" />
+    <parent link="head_xtion_link"/>
+    <child link="head_xtion_depth_frame"/>
+  </joint>
+  <joint name="head_xtion_base_link1" type="fixed" >
+    <origin rpy="0 0 0"
+            xyz="0 -0.045 0" />
+    <parent link="head_xtion_link"/>
+    <child link="head_xtion_rgb_frame"/>
   </joint>
   <joint name="head_xtion_base_link2" type="fixed" >
-        <origin xyz="0 -0.045  0"
-		rpy="0 0 0" />
-	<parent link="head_xtion_link" />
-	<child link="head_xtion_rgb_frame" />
-  </joint>
-  <joint name="head_xtion_base_link3"  type="fixed">
-        <origin xyz="0 0 0"
-		rpy="-1.57 0 1.57" />
-	<parent link="head_xtion_depth_frame" />
-	<child link="head_xtion_depth_optical_frame" />
-  </joint>
-  <joint name="head_xtion_base_link4"  type="fixed">
-        <origin xyz="0 0 0"
-		rpy="-1.57 0 1.57" />
-	<parent link="head_xtion_rgb_frame" />
-	<child link="head_xtion_rgb_optical_frame" />
-  </joint>
--->
+    <origin rpy="-1.5707963267948966 0 -1.5707963267948966"
+            xyz="0 0 0" />
+    <parent link="head_xtion_depth_frame"/>
+    <child link="head_xtion_depth_optical_frame"/>
+  </joint>
+  <joint name="head_xtion_base_link3" type="fixed" >
+    <origin rpy="-1.5707963267948966 0 -1.5707963267948966"
+            xyz="0 0 0" />
+    <parent link="head_xtion_rgb_frame"/>
+    <child link="head_xtion_rgb_optical_frame"/>
+  </joint>
 </robot>

Commit message: using correct frames for xtion

File: scitos_description/urdf/scitos.xacro (robot description, xacro)
@@ -213,5 +213,5 @@
   <link name="head_xtion_link">
     <visual>
-      <origin rpy="0 0 0" xyz="0 0 0"/>
+      <origin rpy="3.14 0 0" xyz="0 0 0"/>
       <geometry>
         <mesh filename="package://scitos_description/meshes/xtion.dae"/>
@@ -331,5 +331,5 @@
   <joint name="head_xtion_base_link" type="fixed" >
     <origin rpy="0 0 0"
-            xyz="0 -0.02 0" />
+            xyz="0 0.045 0" />
     <parent link="head_xtion_link"/>
     <child link="head_xtion_depth_frame"/>
@@ -337,5 +337,5 @@
   <joint name="head_xtion_base_link1" type="fixed" >
     <origin rpy="0 0 0"
-            xyz="0 -0.045 0" />
+            xyz="0 0.02 0" />
     <parent link="head_xtion_link"/>
     <child link="head_xtion_rgb_frame"/>

File: scitos_description/urdf/scitos_calibration.xacro (robot description, xacro)
@@ -20,5 +20,5 @@
   <property name="head_xtion_trans_y" value="0.0" />
   <property name="head_xtion_trans_z" value="0.03" />
-  <property name="head_xtion_rot_x" value="3.14" />
+  <property name="head_xtion_rot_x" value="0" />
   <property name="head_xtion_rot_y" value="0.0" />
   <property name="head_xtion_rot_z" value="0.0" />

Commit message: Added chest camera in urdf model

File: scitos_description/urdf/scitos.xacro (robot description, xacro)
@@ -353,3 +353,53 @@
     <child link="head_xtion_rgb_optical_frame"/>
   </joint>
+  <!-- Connect base to chest_xtion_link -->
+  <link name="chest_xtion_link">
+    <visual>
+      <origin rpy="3.14 0 0" xyz="0 0 0"/>
+      <geometry>
+        <mesh filename="package://scitos_description/meshes/xtion.dae"/>
+      </geometry>
+    </visual>
+    <collision>
+      <origin rpy="0 0 0" xyz="0 0 0.071"/>
+      <geometry>
+        <box size="0.001 0.001 0.001"/>
+      </geometry>
+    </collision>
+  </link>
+  <joint name="chest_xtion_joint" type="fixed" >
+    <!-- Rotation y angle from calibrate_chest and z height from calibrate_chest -->
+    <origin rpy="0 0.72 0" xyz="0.10 0 1.10" />
+    <parent link="base_link"/>
+    <child link="chest_xtion_link"/>
+  </joint>
+  <!-- chest_xtion internal frames -->
+  <link name="chest_xtion_depth_frame"/>
+  <link name="chest_xtion_rgb_frame"/>
+  <link name="chest_xtion_depth_optical_frame"/>
+  <link name="chest_xtion_rgb_optical_frame"/>
+  <joint name="chest_xtion_base_link" type="fixed" >
+    <origin rpy="0 0 0"
+            xyz="0 0.045 0" />
+    <parent link="chest_xtion_link"/>
+    <child link="chest_xtion_depth_frame"/>
+  </joint>
+  <joint name="chest_xtion_base_link1" type="fixed" >
+    <origin rpy="0 0 0"
+            xyz="0 0.02 0" />
+    <parent link="chest_xtion_link"/>
+    <child link="chest_xtion_rgb_frame"/>
+  </joint>
+  <joint name="chest_xtion_base_link2" type="fixed" >
+    <origin rpy="-1.5707963267948966 0 -1.5707963267948966"
+            xyz="0 0 0" />
+    <parent link="chest_xtion_depth_frame"/>
+    <child link="chest_xtion_depth_optical_frame"/>
+  </joint>
+  <joint name="chest_xtion_base_link3" type="fixed" >
+    <origin rpy="-1.5707963267948966 0 -1.5707963267948966"
+            xyz="0 0 0" />
+    <parent link="chest_xtion_rgb_frame"/>
+    <child link="chest_xtion_rgb_optical_frame"/>
+  </joint>
 </robot>

Commit message: Fixed the camera position forward direction

File: scitos_description/urdf/scitos.xacro (robot description, xacro)
@@ -370,5 +370,5 @@
   <joint name="chest_xtion_joint" type="fixed" >
     <!-- Rotation y angle from calibrate_chest and z height from calibrate_chest -->
-    <origin rpy="0 0.72 0" xyz="0.10 0 1.10" />
+    <origin rpy="0 0.72 0" xyz="0.12 0 1.10" />
     <parent link="base_link"/>
     <child link="chest_xtion_link"/>

Commit message: Added broadcaster of chest clibration, does not really work

File: scitos_description/urdf/scitos.xacro (robot description, xacro)
@@ -368,5 +368,5 @@
     </collision>
   </link>
-  <joint name="chest_xtion_joint" type="fixed" >
+  <joint name="chest_xtion_joint" type="continuous" >
     <!-- Rotation y angle from calibrate_chest and z height from calibrate_chest -->
     <origin rpy="0 0.72 0" xyz="0.12 0 1.10" />

Commit message: Got the publisher working now, running it in scitos_state_publisher launch file for ten seconds to update urdf with latest calibration parameters

File: scitos_description/urdf/scitos.xacro (robot description, xacro)
@@ -368,8 +368,18 @@
     </collision>
   </link>
-  <joint name="chest_xtion_joint" type="continuous" >
-    <!-- Rotation y angle from calibrate_chest and z height from calibrate_chest -->
-    <origin rpy="0 0.72 0" xyz="0.12 0 1.10" />
+  <link name="chest_xtion_height_tilt_link"/>
+  <joint name="chest_xtion_height_joint" type="prismatic" >
+    <!-- Z height from calibrate_chest -->
+    <axis xyz="0 0 1"/>
+    <origin rpy="0 0 0" xyz="0.10 0 0" />
+    <limit effort="1000" velocity="1000" lower="0.5" upper="1.5"/>
     <parent link="base_link"/>
+    <child link="chest_xtion_height_tilt_link"/>
+  </joint>
+  <joint name="chest_xtion_tilt_joint" type="continuous" >
+    <!-- Rotation y angle from calibrate_chest-->
+    <axis xyz="0 1 0"/>
+    <origin rpy="0 0 0" xyz="0 0 0" />
+    <parent link="chest_xtion_height_tilt_link"/>
     <child link="chest_xtion_link"/>
   </joint>
@@ -381,5 +391,5 @@
   <joint name="chest_xtion_base_link" type="fixed" >
     <origin rpy="0 0 0"
-            xyz="0 0 0" />
+            xyz="0 0.045 0" />
     <parent link="chest_xtion_link"/>
     <child link="chest_xtion_depth_frame"/>
@@ -387,5 +397,5 @@
   <joint name="chest_xtion_base_link1" type="fixed" >
     <origin rpy="0 0 0"
-            xyz="0 -0.025 0" />
+            xyz="0 0.02 0" />
     <parent link="chest_xtion_link"/>
     <child link="chest_xtion_rgb_frame"/>
